File: EAGLE/MicroWordClock2.sch (EAGLE design)
At the start: 20 parts, among them IC1 ATMEGA328P, IC2 DS1307SMD

Commit message: initial edits to update the existing layout with the same components as the original
Parts:
- removed JP_A, JP_B: (no value), adafruit:PINHD-1X8CLEANBIG
- removed TP_SWITCH, TP_SWITCH_GND: TPB1,27, testpad:TPB1,27
- added J1: (no value), SparkFun-Connectors:USB_AB_SMT
- added R1, R2, R3, R4, R5, R6, R7, R8: 470, SparkFun-Resistors:470OHM-0603-1/10W-1%
- added S2: MOMENTARY-SWITCH-SPST-PTH-RIGHT-ANGLE-KIT, SparkFun-Switches:MOMENTARY-SWITCH-SPST-PTH-RIGHT-ANGLE-KIT
- added U$1, U$10, U$11, U$12, U$13, U$14, U$15, U$16, U$17, U$18, U$19, U$2, U$20, U$21, U$22, U$23, U$24, U$25, U$26, U$27, U$28, U$29, U$3, U$30, U$31, U$32, U$33, U$34, U$35, U$36, U$37, U$38, U$39, U$4, U$40, U$41, U$42, U$43, U$44, U$45, U$46, U$47, U$48, U$49, U$5, U$50, U$51, U$52, U$53, U$54, U$55, U$56, U$57, U$58, U$59, U$6, U$60, U$61, U$62, U$63, U$64, U$7, U$8, U$9: (no value), TULIP_GIZMO:JE2835AWT-00-0000-0B0A0BG840E
Connections:
- removed net A1: IC1.PC1(ADC1), JP_A.1
- removed net A2: IC1.PC0(ADC0), JP_A.2
- removed net A3: IC1.PB2(SS/OC1B), JP_A.3
- removed net A4: IC1.PB1(OC1A), JP_A.4
- removed net A5: IC1.PD5(T1), JP_A.5
- removed net A6: IC1.PB0(ICP), JP_A.6
- removed net A7: IC1.PD6(AIN0), JP_A.7
- removed net A8: IC1.PB7(XTAL2/TOSC2), JP_A.8
- removed net B1: IC1.PC2(ADC2), JP_B.1
- removed net B2: IC1.PC3(ADC3), JP_B.2
- removed net B3: IC1.PD0(RXD), JP_B.3
- removed net B4: IC1.PD1(TXD), JP_B.4
- removed net B5: IC1.PD2(INT0), JP_B.5
- removed net B6: IC1.PD3(INT1), JP_B.6
- removed net B7: IC1.PD4(XCK/T0), JP_B.7
- removed net B8: IC1.PB6(XTAL1/TOSC1), JP_B.8
- new net COL1: IC1.PB1(OC1A), R1.1
- new net COL2: IC1.PD0(RXD), R2.1
- new net COL3: IC1.PD1(TXD), R3.1
- new net COL4: IC1.PD6(AIN0), R4.1
- new net COL5: IC1.PD3(INT1), R5.1
- new net COL6: IC1.PB0(ICP), R6.1
- new net COL7: IC1.PC0(ADC0), R7.1
- new net COL8: IC1.PC1(ADC1), R8.1
- new net EE: R8.2, U$57.C, U$58.C, U$59.C, U$60.C, U$61.C, U$62.C, U$63.C, U$64.C
- new net N$1: S1.1.1
- new net N$11: R1.2, U$1.C, U$2.C, U$3.C, U$4.C, U$5.C, U$6.C, U$7.C, U$8.C
- new net N$15: R2.2, U$10.C, U$11.C, U$12.C, U$13.C, U$14.C, U$15.C, U$16.C, U$9.C
- new net N$5: R3.2, U$17.C, U$18.C, U$19.C, U$20.C, U$21.C, U$22.C, U$23.C, U$24.C
- new net N$6: R4.2, U$25.C, U$26.C, U$27.C, U$28.C, U$29.C, U$30.C, U$31.C, U$32.C
- new net N$7: R5.2, U$33.C, U$34.C, U$35.C, U$36.C, U$37.C, U$38.C, U$39.C, U$40.C
- new net N$8: R6.2, U$41.C, U$42.C, U$43.C, U$44.C, U$45.C, U$46.C, U$47.C, U$48.C
- new net N$9: R7.2, U$49.C, U$50.C, U$51.C, U$52.C, U$53.C, U$54.C, U$55.C, U$56.C
- new net ROW1: IC1.PB7(XTAL2/TOSC2), U$1.A, U$17.A, U$25.A, U$33.A, U$41.A, U$49.A, U$57.A, U$9.A
- new net ROW2: IC1.PB2(SS/OC1B), U$10.A, U$18.A, U$2.A, U$26.A, U$34.A, U$42.A, U$50.A, U$58.A
- new net ROW3: IC1.PB6(XTAL1/TOSC1), U$11.A, U$19.A, U$27.A, U$3.A, U$35.A, U$43.A, U$51.A, U$59.A
- new net ROW4: IC1.PD5(T1), U$12.A, U$20.A, U$28.A, U$36.A, U$4.A, U$44.A, U$52.A, U$60.A
- new net ROW5: IC1.PC2(ADC2), U$13.A, U$21.A, U$29.A, U$37.A, U$45.A, U$5.A, U$53.A, U$61.A
- new net ROW6: IC1.PD4(XCK/T0), U$14.A, U$22.A, U$30.A, U$38.A, U$46.A, U$54.A, U$6.A, U$62.A
- new net ROW7: IC1.PC3(ADC3), U$15.A, U$23.A, U$31.A, U$39.A, U$47.A, U$55.A, U$63.A, U$7.A
- new net ROW8: IC1.PD2(INT0), U$16.A, U$24.A, U$32.A, U$40.A, U$48.A, U$56.A, U$64.A, U$8.A
- net GND: now also J1.SHIELD; no longer TP_SWITCH_GND.TP
- net SWITCH: no longer S1.1.1, TP_SWITCH.TP

Commit message: board with new footprints for switch, microusb and clock & complete routing
Parts:
- removed IC1: ATMEGA328P, atmel:MEGA8-AI
- removed IC2: DS1307SMD, DS1307:DS1307SMD
- removed S2: MOMENTARY-SWITCH-SPST-PTH-RIGHT-ANGLE-KIT, SparkFun-Switches:MOMENTARY-SWITCH-SPST-PTH-RIGHT-ANGLE-KIT
- removed TP_BAT+, TP_BAT-, TP_GND1, TP_VCC1: TPB2,54, testpad:TPB2,54
- removed TP_GND, TP_MISO, TP_MOSI, TP_RST, TP_SCK, TP_VCC: TPB1,27, testpad:TPB1,27
- removed XTAL: XTAL-32KHZ, xtal-32khz:XTAL-32KHZ
- added C3: 4700pF, rcl:C-EUC0603
- added C4: 4.7uF, rcl:C-EUC0603
- added J2: 10118193-0001LF, 10118193-0001LF:10118193-0001LF
- added J3: AVR_SPI_PROG_3X2PTH, SparkFun-Connectors:AVR_SPI_PROG_3X2PTH
- added L1: 120OHM-500MA, OPL_Ferrite_and_Magnetic_Bead:SMD-FERRITE-CHIP-120-OHM-500MA(0603)
- added R9: 10M, rcl:R-EU_R0603
- added U1: ATMEGA328P, atmel:MEGA8-AI
- J1: value (none) -> DS3231S#T&RMODULE; device SparkFun-Connectors:USB_AB_SMT -> DS3231:DS3231S#T&RMODULE
- S1: value SKHMPSE010 -> 1-1825027-1; device switch:SKHMPSE010 -> 1-1825027-1:1-1825027-1
Connections:
- removed net N$14: IC2.X1, XTAL.X2
- removed net N$18: IC1.PC5(ADC5/SCL), IC2.SCL
- removed net N$2: IC2.X2, XTAL.X1
- removed net SWITCH: IC1.PD7(AIN1)
- removed net VBAT: IC2.VBAT, TP_BAT+.TP
- new net PE: C3.2, J2.SHIELD, R9.1
- new net SCL: J1.SDA, U1.PC5(ADC5/SCL)
- new net V_USB: J2.VUSB, L1.1
- net +5V: now also C4.1, J1.VCC, J3.2, L1.2, U1.VCC@1, U1.VCC@2; no longer IC1.VCC@1, IC1.VCC@2, IC2.VCC, TP_VCC.TP, TP_VCC1.TP
- net COL1: now also U1.PB1(OC1A); no longer IC1.PB1(OC1A)
- net COL2: now also U1.PD0(RXD); no longer IC1.PD0(RXD)
- net COL3: now also U1.PD1(TXD); no longer IC1.PD1(TXD)
- net COL4: now also U1.PD6(AIN0); no longer IC1.PD6(AIN0)
- net COL5: now also U1.PD3(INT1); no longer IC1.PD3(INT1)
- net COL6: now also U1.PB0(ICP); no longer IC1.PB0(ICP)
- net COL7: now also U1.PC0(ADC0); no longer IC1.PC0(ADC0)
- net COL8: now also U1.PC1(ADC1); no longer IC1.PC1(ADC1)
- net GND: now also C3.1, C4.2, J1.GND, J2.GND, J2.ID, J3.6, R9.2, S1.2, S1.SHIELD, U1.GND, U1.GND@1, U1.GND@2; no longer IC1.GND, IC1.GND@1, IC1.GND@2, IC2.GND, J1.SHIELD, S1.2.1, S1.2.2, S1.SH, TP_BAT-.TP, TP_GND.TP, TP_GND1.TP
- net MISO: now also J3.1, U1.PB4(MISO); no longer IC1.PB4(MISO), TP_MISO.TP
- net MOSI: now also J3.4, U1.PB3(MOSI/OC2); no longer IC1.PB3(MOSI/OC2), TP_MOSI.TP
- net N$1: now also S1.1, U1.PD7(AIN1); no longer S1.1.1
- net RESET: now also J3.5, U1.PC6(/RESET); no longer IC1.PC6(/RESET), TP_RST.TP
- net ROW1: now also U1.PB7(XTAL2/TOSC2); no longer IC1.PB7(XTAL2/TOSC2)
- net ROW2: now also U1.PB2(SS/OC1B); no longer IC1.PB2(SS/OC1B)
- net ROW3: now also U1.PB6(XTAL1/TOSC1); no longer IC1.PB6(XTAL1/TOSC1)
- net ROW4: now also U1.PD5(T1); no longer IC1.PD5(T1)
- net ROW5: now also U1.PC2(ADC2); no longer IC1.PC2(ADC2)
- net ROW6: now also U1.PD4(XCK/T0); no longer IC1.PD4(XCK/T0)
- net ROW7: now also U1.PC3(ADC3); no longer IC1.PC3(ADC3)
- net ROW8: now also U1.PD2(INT0); no longer IC1.PD2(INT0)
- net SCK: now also J3.3, U1.PB5(SCK); no longer IC1.PB5(SCK), TP_SCK.TP
- net SDA: now also J1.SCL, U1.PC4(ADC4/SDA); no longer IC1.PC4(ADC4/SDA), IC2.SDA
