File: EAGLE/WordClockFace.sch (EAGLE design)
At the start: 4 parts

Commit message: committing the tulip face and fixing a header
Parts:
- J1: device SparkFun-Connectors:CONN_08SMD-STRAIGHT-ALT-FEMALE -> SparkFun-Connectors:CONN_08SMD-STRAIGHT-FEMALE
Changed lines of the file:
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@@
 <?xml version="1.0" encoding="utf-8"?>
 <!DOCTYPE eagle SYSTEM "eagle.dtd">
-<eagle version="9.4.0">
+<eagle version="9.4.2">
 <drawing>
 <settings>
@@
 </classes>
 <parts>
-<part name="J1" library="SparkFun-Connectors" library_urn="urn:adsk.eagle:library:513" deviceset="CONN_08" device="SMD-STRAIGHT-ALT-FEMALE" package3d_urn="urn:adsk.eagle:package:38148/1"/>
+<part name="J1" library="SparkFun-Connectors" library_urn="urn:adsk.eagle:library:513" deviceset="CONN_08" device="SMD-STRAIGHT-FEMALE" package3d_urn="urn:adsk.eagle:package:38144/1"/>
 <part name="J2" library="SparkFun-Connectors" library_urn="urn:adsk.eagle:library:513" deviceset="CONN_08" device="SMD-STRAIGHT-FEMALE" package3d_urn="urn:adsk.eagle:package:38144/1"/>
 <part name="J3" library="SparkFun-Connectors" library_urn="urn:adsk.eagle:library:513" deviceset="CONN_08" device="SMD-STRAIGHT-FEMALE" package3d_urn="urn:adsk.eagle:package:38144/1"/>
